File: minipower.kicad_sch (KiCad schematic)
At the start: 24 parts

Commit message: Added custom footprint and library tables for participants
Parts:
- C1, C2, C3, C4, C5, C6, C7: symbol Device:C -> PCBWorkshop_2026_symbols:C
- D1, D2, D3, D4: symbol Device:D -> PCBWorkshop_2026_symbols:D
- L2: symbol EasyEDA_Lib:SMNR4020-1UH -> PCBWorkshop_2026_symbols:SMNR4020-1UH
- R1, R3, R4, R5, R6, R7, R8: symbol Device:R -> PCBWorkshop_2026_symbols:R
- S1: symbol PCM_JLCPCB-Connectors_Buttons:Tactile Button, 160gf, 12V, 50mA, 4.0mm -> PCBWorkshop_2026_symbols:Tactile Button, 160gf, 12V, 50mA, 4.0mm
- U1: symbol EasyEDA_Lib:IP5306 -> PCBWorkshop_2026_symbols:IP5306
- U2, U3: symbol EasyEDA_Lib:USB-TYPE-C-009 -> PCBWorkshop_2026_symbols:USB-TYPE-C-009
- U6: symbol EasyEDA_Lib:BH-21700-A5BJ001 -> PCBWorkshop_2026_symbols:BH-21700-A5BJ001
Changed lines of the file:
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@@
 	)
 	(symbol
-		(lib_id "power:GND")
+		(lib_id "PCBWorkshop_2026_symbols:GND")
 		(at 172.72 121.92 0)
 		(unit 1)
@@
 	)
 	(symbol
-		(lib_id "Device:R")
+		(lib_id "PCBWorkshop_2026_symbols:R")
 		(at 67.31 102.87 0)
 		(unit 1)
@@
 	)
 	(symbol
-		(lib_id "Device:C")
+		(lib_id "PCBWorkshop_2026_symbols:C")
 		(at 185.42 120.65 0)
 		(unit 1)
@@
 	)
 	(symbol
-		(lib_id "power:GND")
+		(lib_id "PCBWorkshop_2026_symbols:GND")
 		(at 161.29 31.75 180)
 		(unit 1)
@@
 	)
 	(symbol
-		(lib_id "Device:D")
+		(lib_id "PCBWorkshop_2026_symbols:D")
 		(at 124.46 128.27 270)
 		(unit 1)
@@
 	)
 	(symbol
-		(lib_id "Device:R")
+		(lib_id "PCBWorkshop_2026_symbols:R")
 		(at 107.95 43.18 90)
 		(unit 1)
@@
 	)
 	(symbol
-		(lib_id "power:GND")
+		(lib_id "PCBWorkshop_2026_symbols:GND")
 		(at 161.29 52.07 0)
 		(unit 1)
@@
 	)
 	(symbol
-		(lib_id "Device:C")
+		(lib_id "PCBWorkshop_2026_symbols:C")
 		(at 67.31 114.3 0)
 		(unit 1)
@@
 	)
 	(symbol
-		(lib_id "EasyEDA_Lib:BH-21700-A5BJ001")
+		(lib_id "PCBWorkshop_2026_symbols:BH-21700-A5BJ001")
 		(at 210.82 29.21 270)
 		(unit 1)
@@
 	)
 	(symbol
-		(lib_id "EasyEDA_Lib:IP5306")
+		(lib_id "PCBWorkshop_2026_symbols:IP5306")
 		(at 142.24 102.87 0)
 		(unit 1)
@@
 	)
 	(symbol
-		(lib_id "power:GND")
+		(lib_id "PCBWorkshop_2026_symbols:GND")
 		(at 99.06 31.75 180)
 		(unit 1)
@@
 	)
 	(symbol
-		(lib_id "power:GND")
+		(lib_id "PCBWorkshop_2026_symbols:GND")
 		(at 67.31 121.92 0)
 		(unit 1)
@@
 	)
 	(symbol
-		(lib_id "power:GND")
+		(lib_id "PCBWorkshop_2026_symbols:GND")
 		(at 129.54 45.72 0)
 		(unit 1)
@@
 	)
 	(symbol
-		(lib_id "Device:R")
+		(lib_id "PCBWorkshop_2026_symbols:R")
 		(at 107.95 40.64 90)
 		(unit 1)
@@
 	)
 	(symbol
-		(lib_id "power:GND")
+		(lib_id "PCBWorkshop_2026_symbols:GND")
 		(at 185.42 127 0)
 		(unit 1)
@@
 	)
 	(symbol
-		(lib_id "Device:R")
+		(lib_id "PCBWorkshop_2026_symbols:R")
 		(at 163.83 147.32 90)
 		(unit 1)
@@
 	)
 	(symbol
-		(lib_id "power:GND")
+		(lib_id "PCBWorkshop_2026_symbols:GND")
 		(at 210.82 36.83 0)
 		(unit 1)
@@
 	)
 	(symbol
-		(lib_id "power:GND")
+		(lib_id "PCBWorkshop_2026_symbols:GND")
 		(at 142.24 88.9 180)
 		(unit 1)
@@
 	)
 	(symbol
-		(lib_id "Device:D")
+		(lib_id "PCBWorkshop_2026_symbols:D")
 		(at 132.08 128.27 90)
 		(unit 1)
@@
 	)
 	(symbol
-		(lib_id "power:GND")
+		(lib_id "PCBWorkshop_2026_symbols:GND")
 		(at 102.87 110.49 0)
 		(unit 1)
@@
 	)
 	(symbol
-		(lib_id "Device:C")
+		(lib_id "PCBWorkshop_2026_symbols:C")
 		(at 165.1 88.9 0)
 		(unit 1)
@@
 	)
 	(symbol
-		(lib_id "Device:C")
+		(lib_id "PCBWorkshop_2026_symbols:C")
 		(at 172.72 115.57 0)
 		(unit 1)
@@
 	)
 	(symbol
-		(lib_id "EasyEDA_Lib:USB-TYPE-C-009")
+		(lib_id "PCBWorkshop_2026_symbols:USB-TYPE-C-009")
 		(at 82.55 40.64 180)
 		(unit 1)
@@
 	)
 	(symbol
-		(lib_id "Device:C")
+		(lib_id "PCBWorkshop_2026_symbols:C")
 		(at 102.87 102.87 0)
 		(unit 1)
@@
 	)
 	(symbol
-		(lib_id "Device:R")
+		(lib_id "PCBWorkshop_2026_symbols:R")
 		(at 170.18 40.64 90)
 		(unit 1)
@@
 	)
 	(symbol
-		(lib_id "power:GND")
+		(lib_id "PCBWorkshop_2026_symbols:GND")
 		(at 67.31 45.72 0)
 		(unit 1)
@@
 	)
 	(symbol
-		(lib_id "EasyEDA_Lib:SMNR4020-1UH")
+		(lib_id "PCBWorkshop_2026_symbols:SMNR4020-1UH")
 		(at 165.1 105.41 0)
 		(unit 1)
@@
 	)
 	(symbol
-		(lib_id "Device:R")
+		(lib_id "PCBWorkshop_2026_symbols:R")
 		(at 170.18 43.18 90)
 		(unit 1)
@@
 	)
 	(symbol
-		(lib_id "power:GND")
+		(lib_id "PCBWorkshop_2026_symbols:GND")
 		(at 119.38 43.18 0)
 		(unit 1)
@@
 	)
 	(symbol
-		(lib_id "EasyEDA_Lib:USB-TYPE-C-009")
+		(lib_id "PCBWorkshop_2026_symbols:USB-TYPE-C-009")
 		(at 144.78 40.64 180)
 		(unit 1)
@@
 	)
 	(symbol
-		(lib_id "Device:C")
+		(lib_id "PCBWorkshop_2026_symbols:C")
 		(at 190.5 88.9 0)
 		(unit 1)
@@
 	)
 	(symbol
-		(lib_id "PCM_JLCPCB-Connectors_Buttons:Tactile Button, 160gf, 12V, 50mA, 4.0mm")
+		(lib_id "PCBWorkshop_2026_symbols:Tactile Button, 160gf, 12V, 50mA, 4.0mm")
 		(at 179.07 156.21 270)
 		(unit 1)
@@
 	)
 	(symbol
-		(lib_id "power:GND")
+		(lib_id "PCBWorkshop_2026_symbols:GND")
 		(at 187.96 147.32 90)
 		(unit 1)
@@
 	)
 	(symbol
-		(lib_id "power:GND")
+		(lib_id "PCBWorkshop_2026_symbols:GND")
 		(at 190.5 96.52 0)
 		(unit 1)
@@
 	)
 	(symbol
-		(lib_id "Device:D")
+		(lib_id "PCBWorkshop_2026_symbols:D")
 		(at 139.7 128.27 270)
 		(unit 1)
@@
 	)
 	(symbol
-		(lib_id "Device:R")
+		(lib_id "PCBWorkshop_2026_symbols:R")
 		(at 185.42 111.76 0)
 		(unit 1)
@@
 	)
 	(symbol
-		(lib_id "power:GND")
+		(lib_id "PCBWorkshop_2026_symbols:GND")
 		(at 99.06 52.07 0)
 		(unit 1)
@@
 	)
 	(symbol
-		(lib_id "Device:C")
+		(lib_id "PCBWorkshop_2026_symbols:C")
 		(at 177.8 88.9 0)
 		(unit 1)
@@
 	)
 	(symbol
-		(lib_id "Device:D")
+		(lib_id "PCBWorkshop_2026_symbols:D")
 		(at 116.84 128.27 90)
 		(unit 1)

Commit message: add graphic
Other:
- moved on the sheet: C1, C6, R1, R3, S1

Commit message: neatened schematic
Other:
- note added: "Battery"
- note added: "IP5306"
- note added: "Input USB"
- note added: "Output USB"
Changed lines of the file:
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@@
 	(generator_version "9.0")
 	(paper "A4")
+	(rectangle
+		(start 76.2 80.01)
+		(end 209.55 149.86)
+		(stroke
+			(width 0)
+			(type default)
+		)
+		(fill
+			(type none)
+		)
+	)
+	(rectangle
+		(start 125.73 57.15)
+		(end 139.7 60.96)
+		(stroke
+			(width 0)
+			(type default)
+		)
+		(fill
+			(type none)
+		)
+	)
+	(rectangle
+		(start 193.04 57.15)
+		(end 203.2 60.96)
+		(stroke
+			(width 0)
+			(type default)
+		)
+		(fill
+			(type none)
+		)
+	)
+	(rectangle
+		(start 76.2 144.78)
+		(end 86.36 149.86)
+		(stroke
+			(width 0)
+			(type default)
+		)
+		(fill
+			(type none)
+		)
+	)
+	(rectangle
+		(start 59.69 57.15)
+		(end 71.12 60.96)
+		(stroke
+			(width 0)
+			(type default)
+		)
+		(fill
+			(type none)
+		)
+	)
+	(rectangle
+		(start 125.73 22.86)
+		(end 190.5 60.96)
+		(stroke
+			(width 0)
+			(type default)
+		)
+		(fill
+			(type none)
+		)
+	)
+	(rectangle
+		(start 193.04 31.75)
+		(end 209.55 60.96)
+		(stroke
+			(width 0)
+			(type default)
+		)
+		(fill
+			(type none)
+		)
+	)
+	(rectangle
+		(start 59.69 22.86)
+		(end 123.19 60.96)
+		(stroke
+			(width 0)
+			(type default)
+		)
+		(fill
+			(type none)
+		)
+	)
+	(text "IP5306\n"
+		(exclude_from_sim no)
+		(at 81.026 147.828 0)
+		(effects
+			(font
+				(size 1.27 1.27)
+			)
+		)
+	)
+	(text "Battery\n"
+		(exclude_from_sim no)
+		(at 197.866 59.182 0)
+		(effects
+			(font
+				(size 1.27 1.27)
+			)
+		)
+	)
+	(text "Input USB\n"
+		(exclude_from_sim no)
+		(at 65.024 59.436 0)
+		(effects
+			(font
+				(size 1.27 1.27)
+			)
+		)
+	)
+	(text "Output USB\n"
+		(exclude_from_sim no)
+		(at 132.334 59.436 0)
+		(effects
+			(font
+				(size 1.27 1.27)
+			)
+		)
+	)
 	(junction
 		(at 177.8 92.71)
@@
 	(wire
 		(pts
-			(xy 210.82 34.29) (xy 210.82 36.83)
+			(xy 200.66 46.99) (xy 200.66 49.53)
 		)
 		(stroke
@@
 	(wire
 		(pts
-			(xy 210.82 21.59) (xy 210.82 24.13)
+			(xy 200.66 34.29) (xy 200.66 36.83)
 		)
 		(stroke
@@
 	)
 	(label "BAT"
-		(at 210.82 21.59 180)
+		(at 200.66 34.29 180)
 		(effects
 			(font
@@
 		)
 		(instances
-			(project ""
+			(project "minipower"
 				(path "/51d41016-db4f-4152-8650-f97e8de60346"
 					(reference "#PWR04")
@@
 		)
 		(instances
-			(project ""
+			(project "minipower"
 				(path "/51d41016-db4f-4152-8650-f97e8de60346"
 					(reference "R3")
@@
 		)
 		(instances
-			(project ""
+			(project "minipower"
 				(path "/51d41016-db4f-4152-8650-f97e8de60346"
 					(reference "C7")
@@
 		)
 		(instances
-			(project ""
+			(project "minipower"
 				(path "/51d41016-db4f-4152-8650-f97e8de60346"
 					(reference "C6")
@@
 	(symbol
 		(lib_id "PCBWorkshop_2026_symbols:BH-21700-A5BJ001")
-		(at 210.82 29.21 270)
+		(at 200.66 41.91 270)
 		(unit 1)
 		(exclude_from_sim no)
@@
 		(fields_autoplaced yes)
 		(property "Reference" "U6"
-			(at 214.63 27.9399 90)
+			(at 204.47 40.6399 90)
 			(effects
 				(font
@@
 		)
 		(property "Value" "~"
-			(at 214.63 30.4799 90)
+			(at 204.47 43.1799 90)
 			(effects
 				(font
@@
 		)
 		(property "Footprint" "EasyEDA_Lib:BAT-TH_BH-21700-A5BJ001"
-			(at 210.82 29.21 0)
+			(at 200.66 41.91 0)
 			(effects
 				(font
@@
 		)
 		(property "Datasheet" "https://item.szlcsc.com/datasheet/BH-21700-A5BJ001/21949526.html"
-			(at 210.82 29.21 0)
+			(at 200.66 41.91 0)
 			(effects
 				(font
@@
 		)
 		(property "Description" ""
-			(at 210.82 29.21 0)
+			(at 200.66 41.91 0)
 			(effects
 				(font
@@
 		)
 		(property "Manufacturer Part" "BH-21700-A5BJ001"
-			(at 210.82 29.21 0)
+			(at 200.66 41.91 0)
 			(effects
 				(font
@@
 		)
 		(property "Manufacturer" "MYOUNG(美阳)"
-			(at 210.82 29.21 0)
+			(at 200.66 41.91 0)
 			(effects
 				(font
@@
 		)
 		(property "Supplier Part" "C20606809"
-			(at 210.82 29.21 0)
+			(at 200.66 41.91 0)
 			(effects
 				(font
@@
 		)
 		(property "Supplier" "LCSC"
-			(at 210.82 29.21 0)
+			(at 200.66 41.91 0)
 			(effects
 				(font
@@
 		)
 		(property "LCSC Part Name" "BH-21700-A5BJ001"
-			(at 210.82 29.21 0)
+			(at 200.66 41.91 0)
 			(effects
 				(font
@@
 		)
 		(instances
-			(project ""
+			(project "minipower"
 				(path "/51d41016-db4f-4152-8650-f97e8de60346"
 					(reference "U6")
@@
 		)
 		(instances
-			(project ""
+			(project "minipower"
 				(path "/51d41016-db4f-4152-8650-f97e8de60346"
 					(reference "U1")
@@
 		)
 		(instances
-			(project ""
+			(project "minipower"
 				(path "/51d41016-db4f-4152-8650-f97e8de60346"
 					(reference "#PWR012")
@@
 		)
 		(instances
-			(project ""
+			(project "minipower"
 				(path "/51d41016-db4f-4152-8650-f97e8de60346"
 					(reference "#PWR06")
@@
 		)
 		(instances
-			(project ""
+			(project "minipower"
 				(path "/51d41016-db4f-4152-8650-f97e8de60346"
 					(reference "R5")
@@
 		)
 		(instances
-			(project ""
+			(project "minipower"
 				(path "/51d41016-db4f-4152-8650-f97e8de60346"
 					(reference "#PWR03")
@@
 		)
 		(instances
-			(project ""
+			(project "minipower"
 				(path "/51d41016-db4f-4152-8650-f97e8de60346"
 					(reference "R1")
@@
 	(symbol
 		(lib_id "PCBWorkshop_2026_symbols:GND")
-		(at 210.82 36.83 0)
+		(at 200.66 49.53 0)
 		(unit 1)
 		(exclude_from_sim no)
@@
 		(fields_autoplaced yes)
 		(property "Reference" "#PWR09"
-			(at 210.82 43.18 0)
+			(at 200.66 55.88 0)
 			(effects
 				(font
@@
 		)
 		(property "Value" "GND"
-			(at 210.82 41.91 0)
+			(at 200.66 54.61 0)
 			(effects
 				(font
@@
 		)
 		(property "Footprint" ""
-			(at 210.82 36.83 0)
+			(at 200.66 49.53 0)
 			(effects
 				(font
@@
 		)
 		(property "Datasheet" ""
-			(at 210.82 36.83 0)
+			(at 200.66 49.53 0)
 			(effects
 				(font
@@
 		)
 		(property "Description" "Power symbol creates a global label with name \"GND\" , ground"
-			(at 210.82 36.83 0)
+			(at 200.66 49.53 0)
 			(effects
 				(font
@@
 		)
 		(instances
-			(project ""
+			(project "minipower"
 				(path "/51d41016-db4f-4152-8650-f97e8de60346"
 					(reference "#PWR09")
@@
 		)
 		(instances
-			(project ""
+			(project "minipower"
 				(path "/51d41016-db4f-4152-8650-f97e8de60346"
 					(reference "#PWR01")
@@
 		)
 		(instances
-			(project ""
+			(project "minipower"
 				(path "/51d41016-db4f-4152-8650-f97e8de60346"
 					(reference "#PWR07")
@@
 		)
 		(instances
-			(project ""
+			(project "minipower"
 				(path "/51d41016-db4f-4152-8650-f97e8de60346"
 					(reference "C3")
@@
 		)
 		(instances
-			(project ""
+			(project "minipower"
 				(path "/51d41016-db4f-4152-8650-f97e8de60346"
 					(reference "C2")
@@
 		)
 		(instances
-			(project ""
+			(project "minipower"
 				(path "/51d41016-db4f-4152-8650-f97e8de60346"
 					(reference "U2")
@@
 		)
 		(instances
-			(project ""
+			(project "minipower"
 				(path "/51d41016-db4f-4152-8650-f97e8de60346"
 					(reference "C1")
@@
 		)
 		(instances
-			(project ""
+			(project "minipower"
 				(path "/51d41016-db4f-4152-8650-f97e8de60346"
 					(reference "#PWR011")
@@
 		)
 		(instances
-			(project ""
+			(project "minipower"
 				(path "/51d41016-db4f-4152-8650-f97e8de60346"
 					(reference "L2")
@@
 		)
 		(instances
-			(project ""
+			(project "minipower"
 				(path "/51d41016-db4f-4152-8650-f97e8de60346"
 					(reference "#PWR014")
@@
 		)
 		(instances
-			(project ""
+			(project "minipower"
 				(path "/51d41016-db4f-4152-8650-f97e8de60346"
 					(reference "C5")
@@
 		)
 		(instances
-			(project ""
+			(project "minipower"
 				(path "/51d41016-db4f-4152-8650-f97e8de60346"
 					(reference "S1")
@@
 		)
 		(instances
-			(project ""
+			(project "minipower"
 				(path "/51d41016-db4f-4152-8650-f97e8de60346"
 					(reference "#PWR05")
@@
 		)
 		(instances
-			(project ""
+			(project "minipower"
 				(path "/51d41016-db4f-4152-8650-f97e8de60346"
 					(reference "#PWR02")
@@
 		)
 		(instances
-			(project ""
+			(project "minipower"
 				(path "/51d41016-db4f-4152-8650-f97e8de60346"
 					(reference "D4")
@@
 		)
 		(instances
-			(project ""
+			(project "minipower"
 				(path "/51d41016-db4f-4152-8650-f97e8de60346"
 					(reference "R4")
@@
 		)
 		(instances
-			(project ""
+			(project "minipower"
 				(path "/51d41016-db4f-4152-8650-f97e8de60346"
 					(reference "#PWR013")
@@
 		)
 		(instances
-			(project ""
+			(project "minipower"
 				(path "/51d41016-db4f-4152-8650-f97e8de60346"
 					(reference "C4")
@@
 		)
 		(instances
-			(project ""
+			(project "minipower"
 				(path "/51d41016-db4f-4152-8650-f97e8de60346"
 					(reference "D1")
